Commit message: detection and nav

File: src/ugv_gazebo_sim-master/bunker/bunker_description/urdf/bunker.xacro (robot description, xacro)
@@ -4,4 +4,9 @@
      For more information, please see http://wiki.ros.org/sw_urdf_exporter -->
 <robot  name="bunker_description" xmlns:xacro="http://www.ros.org/wiki/xacro">
+      <!-- Xacro arguments for depth camera use -->
+    <xacro:arg name="realsense_enable" default="true" />
+    <xacro:arg name="pointcloud_enable" default="true" />
+     <!-- All Neccesary Header Files, Macros and Constants -->
+  <xacro:include filename="$(find bunker_description)/urdf/includes.xacro" />
   <link
     name="base_link">
@@ -972,4 +977,37 @@
       velocity="0" />
   </joint>
+   <!-- Hokuyo Laser -->
+  <link name="hokuyo_link">
+    <collision>
+      <origin xyz="0 0 0" rpy="0 0 0"/>
+      <geometry>
+    <box size="0.1 0.1 0.1"/>
+      </geometry>
+    </collision>
+    <visual>
+      <origin xyz="0 0 0" rpy="0 0 0"/>
+      <geometry>
+        <mesh filename="package://bunker_description/meshes/hokuyo.dae"/>
+      </geometry>
+    </visual>
+    <inertial>
+      <mass value="1e-5" />
+      <origin xyz="0 0 0" rpy="0 0 Image0"/>
+      <inertia ixx="1e-6" ixy="0" ixz="0" iyy="1e-6" iyz="0" izz="1e-6" />
+    </inertial>
+  </link>
+  <joint name="hokuyo_joint" type="fixed">
+    <axis xyz="0 1 0" />
+    <origin xyz="0.15 0 0.13" rpy="0 0 0"/>
+    <parent link="base_link"/>
+    <child link="hokuyo_link"/>
+  </joint>
+    <!-- REALSENSE CAMERA -->
+      <!-- REALSENSE CAMERA -->
+    <xacro:if value="$(arg realsense_enable)">
+      <xacro:sensor_d435 name="realsense_d435" topics_ns="realsense_d435" parent="base_link" publish_pointcloud="$(arg pointcloud_enable)" >
+        <origin xyz="0.35 0 0.095" rpy="0 0 0" />
+      </xacro:sensor_d435>
+   </xacro:if>
   <!-- /////////////////////////////////   gazebo color   ////////////////////////////////////// -->
  <gazebo reference="base_link">
@@ -985,3 +1023,39 @@
     </plugin>
   </gazebo>
+ <!-- hokuyo -->
+  <gazebo reference="hokuyo_link">
+    <sensor type="gpu_ray" name="head_hokuyo_sensor">
+      <pose>0 0 0 0 0 0</pose>
+      <visualize>false</visualize>
+      <update_rate>40</update_rate>
+      <ray>
+        <scan>
+          <horizontal>
+            <samples>720</samples>
+            <resolution>1</resolution>
+            <min_angle>-2.87979</min_angle>
+            <max_angle>2.87979</max_angle>
+          </horizontal>
+        </scan>
+        <range>
+          <min>0.10</min>
+          <max>30.0</max>
+          <resolution>0.01</resolution>
+        </range>
+        <noise>
+          <type>gaussian</type>
+          <!-- Noise parameters based on published spec for Hokuyo laser
+               achieving "+-30mm" accuracy at range < 10m.  A mean of 0.0m and
+               stddev of 0.01m will put 99.7% of samples within 0.03m of the true
+               reading. -->
+          <mean>0.0</mean>
+          <stddev>0.01</stddev>
+        </noise>
+      </ray>
+      <plugin name="gazebo_ros_head_hokuyo_controller" filename="libgazebo_ros_gpu_laser.so">
+        <topicName>/scan</topicName>
+        <frameName>hokuyo_link</frameName>
+      </plugin>
+    </sensor>
+  </gazebo>
 </robot>

Commit message: buner

File: src/ugv_gazebo_sim-master/bunker/bunker_description/urdf/bunker.xacro (robot description, xacro)
@@ -4,9 +4,4 @@
      For more information, please see http://wiki.ros.org/sw_urdf_exporter -->
 <robot  name="bunker_description" xmlns:xacro="http://www.ros.org/wiki/xacro">
-      <!-- Xacro arguments for depth camera use -->
-    <xacro:arg name="realsense_enable" default="true" />
-    <xacro:arg name="pointcloud_enable" default="true" />
-     <!-- All Neccesary Header Files, Macros and Constants -->
-  <xacro:include filename="$(find bunker_description)/urdf/includes.xacro" />
   <link
     name="base_link">
@@ -977,37 +972,4 @@
       velocity="0" />
   </joint>
-   <!-- Hokuyo Laser -->
-  <link name="hokuyo_link">
-    <collision>
-      <origin xyz="0 0 0" rpy="0 0 0"/>
-      <geometry>
-    <box size="0.1 0.1 0.1"/>
-      </geometry>
-    </collision>
-    <visual>
-      <origin xyz="0 0 0" rpy="0 0 0"/>
-      <geometry>
-        <mesh filename="package://bunker_description/meshes/hokuyo.dae"/>
-      </geometry>
-    </visual>
-    <inertial>
-      <mass value="1e-5" />
-      <origin xyz="0 0 0" rpy="0 0 Image0"/>
-      <inertia ixx="1e-6" ixy="0" ixz="0" iyy="1e-6" iyz="0" izz="1e-6" />
-    </inertial>
-  </link>
-  <joint name="hokuyo_joint" type="fixed">
-    <axis xyz="0 1 0" />
-    <origin xyz="0.15 0 0.13" rpy="0 0 0"/>
-    <parent link="base_link"/>
-    <child link="hokuyo_link"/>
-  </joint>
-    <!-- REALSENSE CAMERA -->
-      <!-- REALSENSE CAMERA -->
-    <xacro:if value="$(arg realsense_enable)">
-      <xacro:sensor_d435 name="realsense_d435" topics_ns="realsense_d435" parent="base_link" publish_pointcloud="$(arg pointcloud_enable)" >
-        <origin xyz="0.35 0 0.095" rpy="0 0 0" />
-      </xacro:sensor_d435>
-   </xacro:if>
   <!-- /////////////////////////////////   gazebo color   ////////////////////////////////////// -->
  <gazebo reference="base_link">
@@ -1023,39 +985,3 @@
     </plugin>
   </gazebo>
- <!-- hokuyo -->
-  <gazebo reference="hokuyo_link">
-    <sensor type="gpu_ray" name="head_hokuyo_sensor">
-      <pose>0 0 0 0 0 0</pose>
-      <visualize>false</visualize>
-      <update_rate>40</update_rate>
-      <ray>
-        <scan>
-          <horizontal>
-            <samples>720</samples>
-            <resolution>1</resolution>
-            <min_angle>-2.87979</min_angle>
-            <max_angle>2.87979</max_angle>
-          </horizontal>
-        </scan>
-        <range>
-          <min>0.10</min>
-          <max>30.0</max>
-          <resolution>0.01</resolution>
-        </range>
-        <noise>
-          <type>gaussian</type>
-          <!-- Noise parameters based on published spec for Hokuyo laser
-               achieving "+-30mm" accuracy at range < 10m.  A mean of 0.0m and
-               stddev of 0.01m will put 99.7% of samples within 0.03m of the true
-               reading. -->
-          <mean>0.0</mean>
-          <stddev>0.01</stddev>
-        </noise>
-      </ray>
-      <plugin name="gazebo_ros_head_hokuyo_controller" filename="libgazebo_ros_gpu_laser.so">
-        <topicName>/scan</topicName>
-        <frameName>hokuyo_link</frameName>
-      </plugin>
-    </sensor>
-  </gazebo>
 </robot>
